File: probador-motores-pap/control-probador-motores-pap/control-probador-motores-pap.kicad_pcb (KiCad board)
At the start: 2 copper layers, 50 x 35 mm, 11 parts, among them J1 Screw_Terminal_01x06, P1 SW_Push, U1 NE555

Commit message: Add files via upload
Parts:
- moved R1 4.27 mm to (133.9, 87.3)
- moved S1 2.37 mm to (108.5, 70.5)
- moved P1 2.31 mm to (130.0, 70.5)
- moved S2 2.30 mm to (118.5, 70.5)
- moved C1 1.77 mm to (108.7, 100.5)
- moved C3 0.97 mm to (122.0, 93.5)
- moved C2 0.87 mm to (128.4, 93.5)
Routing:
- net Net-(R1-Pad2): track 26.6 -> 32.4 mm
- net Net-(C2-Pad1): track 37.8 -> 33.4 mm
- net Net-(R2-Pad2): track 20.3 -> 22.2 mm
- net /Reloj: track 30.3 -> 28.7 mm
- net +5V: track 144.7 -> 143.3 mm
- net /Medio_Full_Paso: track 39.1 -> 40.0 mm
- net Net-(C3-Pad1): track 3.23 -> 4.16 mm
- net /Direccion: track 25.1 -> 25.9 mm
- removed copper zone on B.Cu, net +5V
- removed copper zone on B.Cu, net GND
- removed copper zone on B.Cu, net Net-(C2-Pad1)
Other:
- board size 50 x 35 mm -> 51 x 37 mm
- net class CNC added: clearance 0.5, trace_width 1, via_dia 0.8, via_drill 0.4
- net class Default: clearance 0.2 -> 0.3
- rule solder_mask_min_width: 0.25 -> 0.5
- rule trace_clearance: 0.2 -> 0.3

Commit message: Add files via upload
Parts:
- moved C2 15.1 mm to (115.0, 100.5), turned to 0 degrees
- moved C3 14.6 mm to (108.5, 99.0), turned to 180 degrees
- moved U1 10.4 mm to (119.2, 82.5)
- moved C1 8.83 mm to (101.2, 105.2)
- moved RV1 7.69 mm to (99.8, 92.8)
- moved S1 6.50 mm to (102.0, 70.5)
- moved R1 5.41 mm to (128.5, 87.8)
- moved S2 4.25 mm to (114.2, 70.5)
- moved R2 4.11 mm to (121.5, 94.2), turned to 180 degrees
- moved P1 3.25 mm to (126.8, 70.5)
Routing:
- net GND: track 54.0 -> 88.5 mm
- net +5V: track 143.3 -> 177.6 mm
- net Net-(R2-Pad2): track 22.2 -> 7.13 mm
- net Net-(R1-Pad2): track 32.4 -> 19.8 mm
- net /Reloj: track 28.7 -> 36.4 mm
- net Net-(C3-Pad1): track 4.16 -> 10.2 mm
- net /Direccion: track 25.9 -> 30.0 mm
- net /Medio_Full_Paso: track 40.0 -> 43.6 mm
- net /Permitir: track 11.4 -> 14.6 mm
- net Net-(C2-Pad1): track 33.4 -> 36.0 mm
Other:
- board size 51 x 37 mm -> 60 x 40 mm
- net class CNC: trace_width 1 -> 1.2; via_dia 0.8 -> 1; via_drill 0.4 -> 0.5
- net class Default: clearance 0.3 -> 0.5; trace_width 0.25 -> 2; via_dia 0.8 -> 1; via_drill 0.4 -> 0.5
- rule trace_clearance: 0.3 -> 0.5
- rule via_min_size: 0.4 -> 0.8
