File: probador-motores-pap/control-probador-motores-pap/control-probador-motores-pap.sch (KiCad schematic (older format))
At the start: 11 parts, among them J1 Screw_Terminal_01x06, P1 SW_Push, U1 NE555

Commit message: Add files via upload
Changed lines of the file:
@@
 	6150 3200 6150 3050
 Wire Wire Line
-	6150 2550 6850 2550
+	6150 2550 6350 2550
 Wire Wire Line
 	7700 2800 7700 2550
@@
 	8450 3700 7750 3700
 Wire Wire Line
-	7750 3700 7750 4700
+	7750 3700 7750 4400
 $Comp
 L power:GND #PWR0104
@@
 Wire Wire Line
 	5900 2550 5600 2550
+$Comp
+L power:PWR_FLAG #FLG0101
+U 1 1 606AF1B0
+P 6350 2400
+F 0 "#FLG0101" H 6350 2475 50  0001 C CNN
+F 1 "PWR_FLAG" H 6350 2573 50  0000 C CNN
+F 2 "" H 6350 2400 50  0001 C CNN
+F 3 "~" H 6350 2400 50  0001 C CNN
+	1    6350 2400
+	1    0    0    -1
+$EndComp
+$Comp
+L power:PWR_FLAG #FLG0102
+U 1 1 606AF931
+P 7200 4200
+F 0 "#FLG0102" H 7200 4275 50  0001 C CNN
+F 1 "PWR_FLAG" H 7200 4373 50  0000 C CNN
+F 2 "" H 7200 4200 50  0001 C CNN
+F 3 "~" H 7200 4200 50  0001 C CNN
+	1    7200 4200
+	1    0    0    -1
+$EndComp
+Wire Wire Line
+	7200 4200 7200 4400
+Wire Wire Line
+	7200 4400 7750 4400
+Connection ~ 7750 4400
+Wire Wire Line
+	7750 4400 7750 4700
+Wire Wire Line
+	6350 2400 6350 2550
+Connection ~ 6350 2550
+Wire Wire Line
+	6350 2550 6850 2550
 $EndSCHEMATC
